Commit message: astra placement, m8 placement

File: turtlebot_description/urdf/sensors/astra.urdf.xacro (robot description, xacro)
@@ -4,14 +4,31 @@
   <xacro:include filename="$(find turtlebot_description)/urdf/turtlebot_properties.urdf.xacro"/>
   <!-- Xacro properties -->
-  <xacro:property name="astra_cam_py" value="-0.0125"/>
+  <xacro:property name="astra_cam_px" value="-0.102"/> <!-- ${cam_px} -->
+  <xacro:property name="astra_cam_py" value="0"/>
+  <xacro:property name="astra_cam_pz" value="0.281"/> <!-- ${cam_pz} -->
   <xacro:property name="astra_depth_rel_rgb_py" value="0.0250" />
   <xacro:property name="astra_cam_rel_rgb_py"   value="-0.0125" />
-  <xacro:property name="astra_dae_display_scale"   value="1" />
+  <xacro:property name="astra_dae_display_scale"   value=".001" />
   <!-- Parameterised in part by the values in turtlebot_properties.urdf.xacro -->
   <xacro:macro name="sensor_astra" params="parent">
+    <joint name="astra_mount" type="fixed">
+      <origin xyz="${astra_cam_px} ${astra_cam_py} ${astra_cam_pz}"
+        rpy="0 0 ${M_PI/2}"/>
+      <parent link="${parent}"/>
+      <child link="astra_mount_joint"/>
+    </joint>
+    <link name="astra_mount_joint">
+      <visual>
+        <origin xyz="0 0 0" rpy="0 0 0"/>
+        <geometry>
+          <mesh filename="package://turtlebot_description/meshes/sensors/astra_mount.STL" scale="${astra_dae_display_scale} ${astra_dae_display_scale} ${astra_dae_display_scale}"/>
+        </geometry>
+        <xacro:insert_block name="material_dark_grey" />
+      </visual>
+    </link>
     <joint name="camera_rgb_joint" type="fixed">
-      <origin xyz="${cam_px} ${astra_cam_py} ${cam_pz}"
+      <origin xyz="0 0 0 "
               rpy="0 0 0"/>
-      <parent link="${parent}"/>
+      <parent link="astra_mount_joint"/>
       <child link="camera_rgb_frame" />
     </joint>
@@ -31,8 +48,9 @@
     <link name="camera_link">
       <visual>
-        <origin xyz="-0.04 0.02 -0.01" rpy="${M_PI/2} 0 ${M_PI/2}"/>
+        <origin xyz="0 .021 0" rpy="0 0 0"/>
         <geometry>
-          <mesh filename="package://turtlebot_description/meshes/sensors/astra.dae" scale="${astra_dae_display_scale} ${astra_dae_display_scale} ${astra_dae_display_scale}"/>
+          <mesh filename="package://turtlebot_description/meshes/sensors/astra.STL" scale="${astra_dae_display_scale} ${astra_dae_display_scale} ${astra_dae_display_scale}"/>
         </geometry>
+        <xacro:insert_block name="material_black" />
       </visual>
       <collision>

Commit message: rotate 3d models

File: turtlebot_description/urdf/sensors/astra.urdf.xacro (robot description, xacro)
@@ -14,5 +14,5 @@
     <joint name="astra_mount" type="fixed">
       <origin xyz="${astra_cam_px} ${astra_cam_py} ${astra_cam_pz}"
-        rpy="0 0 ${M_PI/2}"/>
+        rpy="0 0 0"/>
       <parent link="${parent}"/>
       <child link="astra_mount_joint"/>
@@ -20,5 +20,5 @@
     <link name="astra_mount_joint">
       <visual>
-        <origin xyz="0 0 0" rpy="0 0 0"/>
+        <origin xyz="0 0 0" rpy="0 0 ${M_PI/2}"/>
         <geometry>
           <mesh filename="package://turtlebot_description/meshes/sensors/astra_mount.STL" scale="${astra_dae_display_scale} ${astra_dae_display_scale} ${astra_dae_display_scale}"/>
@@ -48,5 +48,5 @@
     <link name="camera_link">
       <visual>
-        <origin xyz="0 .021 0" rpy="0 0 0"/>
+        <origin xyz="0 .021 0" rpy="0 0 ${M_PI/2}"/>
         <geometry>
           <mesh filename="package://turtlebot_description/meshes/sensors/astra.STL" scale="${astra_dae_display_scale} ${astra_dae_display_scale} ${astra_dae_display_scale}"/>
